File: PowerMod.kicad_sch (KiCad schematic)
At the start: 7 parts, among them J1 Conn_01x12_Pin, J2 Conn_01x12_Pin, U1 L7805

Commit message: Fix wrong U1 footprint, improve silkscreen
Connections:
- net GNDPWR: now also U1.3 (GND); no longer U1.2 (GND)
- net at D1.2 (A): now also U1.2 (OUT); no longer U1.3 (OUT)
Other:
- moved on the sheet: U1
Changed lines of the file:
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@@
+	)
+	(junction
+		(at 134.62 82.55)
+		(diameter 0)
+		(color 0 0 0 0)
 	)
 	(junction
@@
 	)
 	(junction
-		(at 134.62 82.55)
+		(at 124.46 87.63)
 		(diameter 0)
 		(color 0 0 0 0)
@@
 	)
 	(junction
-		(at 124.46 91.44)
-		(diameter 0)
-		(color 0 0 0 0)
-	)
-	(junction
 		(at 151.13 99.06)
 		(diameter 0)
@@
 	(wire
 		(pts
+			(xy 132.08 96.52) (xy 137.16 96.52)
+		)
+		(stroke
+			(width 0)
+			(type default)
+		)
+	)
+	(wire
+		(pts
 			(xy 153.67 96.52) (xy 151.13 96.52)
 		)
@@
 	(wire
 		(pts
+			(xy 124.46 104.14) (xy 134.62 104.14)
+		)
+		(stroke
+			(width 0)
+			(type default)
+		)
+	)
+	(wire
+		(pts
 			(xy 151.13 77.47) (xy 153.67 77.47)
 		)
@@
 	(wire
 		(pts
-			(xy 134.62 101.6) (xy 134.62 99.06)
-		)
-		(stroke
-			(width 0)
-			(type default)
-		)
-	)
-	(wire
-		(pts
 			(xy 151.13 99.06) (xy 151.13 101.6)
 		)
@@
 	(wire
 		(pts
+			(xy 134.62 104.14) (xy 134.62 82.55)
+		)
+		(stroke
+			(width 0)
+			(type default)
+		)
+	)
+	(wire
+		(pts
 			(xy 151.13 101.6) (xy 153.67 101.6)
 		)
@@
 	(wire
 		(pts
+			(xy 124.46 87.63) (xy 124.46 88.9)
+		)
+		(stroke
+			(width 0)
+			(type default)
+		)
+	)
+	(wire
+		(pts
 			(xy 151.13 59.69) (xy 153.67 59.69)
 		)
@@
 	(wire
 		(pts
-			(xy 124.46 91.44) (xy 127 91.44)
-		)
-		(stroke
-			(width 0)
-			(type default)
-		)
-	)
-	(wire
-		(pts
 			(xy 151.13 62.23) (xy 153.67 62.23)
 		)
@@
 	(wire
 		(pts
-			(xy 137.16 101.6) (xy 134.62 101.6)
-		)
-		(stroke
-			(width 0)
-			(type default)
-		)
-	)
-	(wire
-		(pts
 			(xy 134.62 74.93) (xy 138.43 74.93)
 		)
@@
 	(wire
 		(pts
-			(xy 124.46 82.55) (xy 124.46 91.44)
-		)
-		(stroke
-			(width 0)
-			(type default)
-		)
-	)
-	(wire
-		(pts
-			(xy 134.62 83.82) (xy 134.62 82.55)
+			(xy 124.46 82.55) (xy 124.46 87.63)
 		)
 		(stroke
@@
 	(wire
 		(pts
+			(xy 137.16 96.52) (xy 137.16 101.6)
+		)
+		(stroke
+			(width 0)
+			(type default)
+		)
+	)
+	(wire
+		(pts
 			(xy 151.13 101.6) (xy 151.13 104.14)
 		)
@@
 	(wire
 		(pts
-			(xy 123.19 91.44) (xy 124.46 91.44)
+			(xy 123.19 87.63) (xy 124.46 87.63)
 		)
 		(stroke
@@
 	(symbol
 		(lib_id "Regulator_Linear:L7805")
-		(at 134.62 91.44 270)
+		(at 124.46 96.52 90)
 		(unit 1)
 		(exclude_from_sim no)
@@
 		(fields_autoplaced yes)
 		(property "Reference" "U1"
-			(at 138.43 90.1699 90)
+			(at 120.65 95.2499 90)
 			(effects
 				(font
@@
 		)
 		(property "Value" "L7805"
-			(at 138.43 92.7099 90)
+			(at 120.65 97.7899 90)
 			(effects
 				(font
@@
 		)
 		(property "Footprint" "Custom:VREG_L7805CDT-TR"
-			(at 130.81 92.075 0)
+			(at 132.842 82.296 0)
 			(effects
 				(font
@@
 		)
 		(property "Datasheet" "http://www.st.com/content/ccc/resource/technical/document/datasheet/41/4f/b3/b0/12/d4/47/88/CD00000444.pdf/files/CD00000444.pdf/jcr:content/translations/en.CD00000444.pdf"
-			(at 133.35 91.44 0)
+			(at 144.526 96.52 0)
 			(effects
 				(font
@@
 		)
 		(property "Description" "Positive 1.5A 35V Linear Regulator, Fixed Output 5V, TO-220/TO-263/TO-252"
-			(at 134.62 91.44 0)
+			(at 150.114 97.536 0)
 			(effects
 				(font
@@
 	(symbol
 		(lib_id "power:GNDPWR")
-		(at 123.19 91.44 270)
+		(at 123.19 87.63 270)
 		(unit 1)
 		(exclude_from_sim no)
@@
 		(fields_autoplaced yes)
 		(property "Reference" "#PWR01"
-			(at 118.11 91.44 0)
+			(at 118.11 87.63 0)
 			(effects
 				(font
@@
 		)
 		(property "Value" "GNDPWR"
-			(at 119.38 91.3129 90)
+			(at 119.38 87.5029 90)
 			(effects
 				(font
@@
 		)
 		(property "Footprint" ""
-			(at 121.92 91.44 0)
+			(at 121.92 87.63 0)
 			(effects
 				(font
@@
 		)
 		(property "Datasheet" ""
-			(at 121.92 91.44 0)
+			(at 121.92 87.63 0)
 			(effects
 				(font
@@
 		)
 		(property "Description" "Power symbol creates a global label with name \"GNDPWR\" , global ground"
-			(at 123.19 91.44 0)
-			(effects
-				(font
+			(at 123.19 87.63 0)
+			(effects
+				(font

Commit message: Updated TVS diode
Parts:
- D2: value TVS 29.2V -> SMBJ36A
Changed lines of the file:
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@@
 			)
 		)
-		(property "Value" "TVS 29.2V"
+		(property "Value" "SMBJ36A"
 			(at 142.24 71.12 0)
 			(effects

Commit message: Updated schematic to be much clearer
Connections:
- net OUT+: now reaches C2.1, D1.1 (K), J2.10 (Pin_10), J2.11 (Pin_11), J2.12 (Pin_12), J2.8 (Pin_8), J2.9 (Pin_9)
- net IN+: now reaches C1.1, D2.1 (K), J1.10 (Pin_10), J1.11 (Pin_11), J1.12 (Pin_12), J1.8 (Pin_8), J1.9 (Pin_9), U1.1 (IN)
Other:
- moved on the sheet: C1, C2, D1, D2, J1, J2, U1

Commit message: Complete re-design
Parts:
- removed C1: 1uf, Custom:CAPMP3.7X2.8_2.1N_KEM, symbol Device:C_Polarized
- removed C2: 330mf, Custom:CAP_20SVPK68M, symbol Device:C_Polarized
- removed D1: B160-E3, Diode_SMD:D_SMA, symbol Diode:B160-E3
- removed D2: SMBJ36A, Custom:DIOM4336X265N, symbol Device:D_Zener
- removed U1: L7805, Custom:VREG_L7805CDT-TR, symbol Regulator_Linear:L7805
- added C1: 1uf, Capacitor_SMD:C_1206_3216Metric, symbol SymbolLib2:C
- added C2: 10uf, Capacitor_SMD:C_1206_3216Metric, symbol SymbolLib2:C
- added C4, C5, C6, C7: 33uf, Capacitor_SMD:C_1206_3216Metric, symbol SymbolLib2:C
- added D1: B160-E3, Diode_SMD:D_SMA, symbol SymbolLib2:B160-E3
- added D2: LED, LED_SMD:LED_0805_2012Metric, symbol SymbolLib2:LED
- added R1: 400, Resistor_SMD:R_1206_3216Metric, symbol SymbolLib2:R
- added U1: TPS7B8650DQDDARQ1, Footprints:DDA0008B-IPC_B, symbol SymbolLib2:TPS7B8650DQDDARQ1
- J1, J2: symbol Connector:Conn_01x12_Pin -> SymbolLib2:Conn_01x12_Pin
Connections:
- net GNDPWR: now also C1.1, C2.1, C4.2, C5.2, C6.2, C7.2, R1.1, U1.5 (GND), U1.9 (Thermal_Pad)
- net IN+: now also C1.2, U1.7 (EN), U1.8 (IN)
- net OUT+: now also C4.1, C5.1, C6.1, C7.1, D1.1 (K)
- new net: C2.2, D1.2 (A), D2.2 (A), U1.1 (OUT)
- new net: D2.1 (K), R1.2
Other:
- moved on the sheet: J1, J2
