File: PowerMod.kicad_sch (KiCad schematic)
At the start: 7 parts, among them J1 Conn_01x12_Pin, J2 Conn_01x12_Pin, U1 L7805

Commit message: Embedded symbols and footprints
Parts:
- C1, C2: symbol Device:C_Polarized -> SymLibrary:C_Polarized
- D1: symbol Diode:B160-E3 -> SymLibrary:B160-E3
- D2: symbol Device:D_Zener -> SymLibrary:D_Zener
- J1, J2: symbol Connector:Conn_01x12_Pin -> SymLibrary:Conn_01x12_Pin
- U1: symbol Regulator_Linear:L7805 -> SymLibrary:L7805
Changed lines of the file:
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@@
 	)
 	(symbol
-		(lib_id "Connector:Conn_01x12_Pin")
+		(lib_id "SymLibrary:Conn_01x12_Pin")
 		(at 41.91 31.75 180)
 		(unit 1)
@@
 	)
 	(symbol
-		(lib_id "power:GNDPWR")
+		(lib_id "SymLibrary:GNDPWR")
 		(at 111.76 104.14 0)
 		(unit 1)
@@
 	)
 	(symbol
-		(lib_id "power:GNDPWR")
+		(lib_id "SymLibrary:GNDPWR")
 		(at 121.92 72.39 90)
 		(unit 1)
@@
 	)
 	(symbol
-		(lib_id "Regulator_Linear:L7805")
+		(lib_id "SymLibrary:L7805")
 		(at 111.76 72.39 0)
 		(unit 1)
@@
 	)
 	(symbol
-		(lib_id "Device:C_Polarized")
+		(lib_id "SymLibrary:C_Polarized")
 		(at 111.76 99.06 0)
 		(unit 1)
@@
 	)
 	(symbol
-		(lib_id "power:GNDPWR")
+		(lib_id "SymLibrary:GNDPWR")
 		(at 29.21 39.37 270)
 		(unit 1)
@@
 	)
 	(symbol
-		(lib_id "Connector:Conn_01x12_Pin")
+		(lib_id "SymLibrary:Conn_01x12_Pin")
 		(at 41.91 76.2 180)
 		(unit 1)
@@
 	)
 	(symbol
-		(lib_id "Device:D_Zener")
+		(lib_id "SymLibrary:D_Zener")
 		(at 90.17 64.77 90)
 		(unit 1)
@@
 	)
 	(symbol
-		(lib_id "power:GNDPWR")
+		(lib_id "SymLibrary:GNDPWR")
 		(at 93.98 57.15 180)
 		(unit 1)
@@
 	)
 	(symbol
-		(lib_id "Device:C_Polarized")
+		(lib_id "SymLibrary:C_Polarized")
 		(at 97.79 64.77 180)
 		(unit 1)
@@
 	)
 	(symbol
-		(lib_id "Diode:B160-E3")
+		(lib_id "SymLibrary:B160-E3")
 		(at 111.76 86.36 90)
 		(unit 1)
@@
 	)
 	(symbol
-		(lib_id "power:GNDPWR")
+		(lib_id "SymLibrary:GNDPWR")
 		(at 33.02 83.82 270)
 		(unit 1)
