File: PowerMod.kicad_pcb (KiCad board)
At the start: 2 copper layers, 16.2 x 23.8 mm, 7 parts, among them J1 Conn_01x12_Pin, J2 Conn_01x12_Pin, U1 L7805

Commit message: Fix wrong U1 footprint, improve silkscreen
Parts:
- moved D1 0.68 mm to (119.5, 96.3)
Connections:
- U1 pad 2: GNDPWR -> Net-(D1-A)
- U1 pad 3: Net-(D1-A) -> GNDPWR
Routing:
- net GNDPWR: track 14.7 -> 12.4 mm, vias 1 -> 6
- net Net-(D1-A): track 8.07 -> 9.93 mm
- net Net-(D1-K): track 19.4 -> 18.7 mm
Other:
- board text added: "Heatsink required"
- board text added: "Nanoka DC-DC Module Input: 6v min, 2Ov max Output: 5v @ 1.5A max"
- board text added: "OUT"
- board text removed: "Nanoka DC-DC Module Input: 6v min, 14v max Output: 5v @ 500 mAH max"
Changed lines of the file:
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@@
 			(drillshape 0)
 			(scaleselection 1)
-			(outputdirectory "../../../../Desktop/PCBs/NanokaPowerMod/")
+			(outputdirectory "/home/miohatsume/Desktop/PCBs/NanokaPowerMod/v2/")
 		)
 	)
@@
 			(layer "F.SilkS")
 		)
-		(fp_circle
-			(center -4 0)
-			(end -3.9 0)
-			(stroke
-				(width 0.2)
-				(type solid)
-			)
-			(fill no)
-			(layer "F.SilkS")
-		)
 		(fp_line
 			(start 3.555 2.0625)
@@
 				(type solid)
 			)
-			(layer "F.Fab")
-		)
-		(fp_circle
-			(center -4 0)
-			(end -3.9 0)
-			(stroke
-				(width 0.2)
-				(type solid)
-			)
-			(fill no)
 			(layer "F.Fab")
 		)
@@
 		(at 127.5 94.47)
 		(property "Reference" "U1"
-			(at 0 3.53 0)
+			(at 0 1.93 0)
 			(layer "F.SilkS")
 			(effects
@@
 			(layer "F.SilkS")
 		)
-		(fp_circle
-			(center -3.786 3.9)
-			(end -3.686 3.9)
-			(stroke
-				(width 0.127)
-				(type solid)
-			)
-			(fill no)
-			(layer "F.SilkS")
-		)
 		(fp_line
 			(start -3.55 -5.65)
@@
 				(type solid)
 			)
-			(layer "F.Fab")
-		)
-		(fp_circle
-			(center -3.786 3.9)
-			(end -3.686 3.9)
-			(stroke
-				(width 0.127)
-				(type solid)
-			)
-			(fill no)
 			(layer "F.Fab")
 		)
@@
 			(size 0.98 2.4)
 			(layers "F.Cu" "F.Mask" "F.Paste")
+			(net 8 "Net-(D1-A)")
+			(pinfunction "OUT")
+			(pintype "power_out")
+			(solder_mask_margin 0.102)
+		)
+		(pad "3" smd rect
+			(at 0 -2.47)
+			(size 5.86 5.57)
+			(layers "F.Cu" "F.Mask")
 			(net 6 "GNDPWR")
 			(pinfunction "GND")
@@
 			(solder_mask_margin 0.102)
 		)
-		(pad "3" smd rect
-			(at 0 -2.47)
-			(size 5.86 5.57)
-			(layers "F.Cu" "F.Mask")
-			(net 8 "Net-(D1-A)")
-			(pinfunction "OUT")
-			(pintype "power_out")
-			(solder_mask_margin 0.102)
-		)
 		(embedded_fonts no)
 		(model "/home/miohatsume/Documents/KiCad Custom Libraries/3D Models/L7805CDT-TR.step"
@@
 			(layer "F.SilkS")
 		)
-		(fp_circle
-			(center -3.55 -1.5)
-			(end -3.45 -1.5)
-			(stroke
-				(width 0.2)
-				(type solid)
-			)
-			(fill no)
-			(layer "F.SilkS")
-		)
 		(fp_line
 			(start 3.95 1.05)
@@
 				(type solid)
 			)
-			(layer "F.Fab")
-		)
-		(fp_circle
-			(center -3.55 -1.5)
-			(end -3.45 -1.5)
-			(stroke
-				(width 0.2)
-				(type solid)
-			)
-			(fill no)
 			(layer "F.Fab")
 		)
@@
 	(footprint "Diode_SMD:D_SMA"
 		(layer "F.Cu")
-		(at 119.5 97)
+		(at 119.475 96.325)
 		(descr "Diode SMA (DO-214AC)")
 		(tags "Diode SMA (DO-214AC)")
@@
 	)
 	(gr_rect
+		(start 121.821675 101.175)
+		(end 122.178325 101.874998)
+		(stroke
+			(width 0.1)
+			(type solid)
+		)
+		(fill yes)
+		(layer "F.SilkS")
+	)
+	(gr_line
+		(start 121.5 97.975)
+		(end 121.5 97.275)
+		(stroke
+			(width 0.1)
+			(type default)
+		)
+		(layer "F.SilkS")
+	)
+	(gr_rect
+		(start 115.915 94.675)
+		(end 116.15 97.975)
+		(stroke
+			(width 0.1)
+			(type solid)
+		)
+		(fill yes)
+		(layer "F.SilkS")
+	)
+	(gr_rect
+		(start 125.946005 105.061502)
+		(end 129.05 105.288498)
+		(stroke
+			(width 0.1)
+			(type solid)
+		)
+		(fill yes)
+		(layer "F.SilkS")
+	)
+	(gr_rect
+		(start 121.80585 104.1125)
+		(end 122.1625 104.8125)
+		(stroke
+			(width 0.1)
+			(type solid)
+		)
+		(fill yes)
+		(layer "F.SilkS")
+	)
+	(gr_line
+		(start 121.475 95.375)
+		(end 121.475 94.675)
+		(stroke
+			(width 0.1)
+			(type default)
+		)
+		(layer "F.SilkS")
+	)
+	(gr_poly
+		(pts
+			(xy 122.85 88.525) (xy 123.85 88.525) (xy 123.35 88.025)
+		)
+		(stroke
+			(width 0.1)
+			(type solid)
+		)
+		(fill yes)
+		(layer "B.SilkS")
+	)
+	(gr_rect
 		(start 115.305 85.1125)
 		(end 131.5 108.8875)
@@
 		(layer "Edge.Cuts")
 	)
-	(gr_text "Nanoka DC-DC Module\nInput: 6v min, 14v max\nOutput: 5v @ 500 mAH max"
-		(at 127 91 0)
+	(gr_text "Nanoka DC-DC Module\nInput: 6v min, 2Ov max\nOutput: 5v @ 1.5A max "
+		(at 127.35 98.225 0)
 		(layer "B.SilkS")
 		(effects
@@
 		)
 	)
+	(gr_text "Heatsink required"
+		(at 126.5 99.6 0)
+		(layer "B.SilkS")
+		(effects
+			(font
+				(size 0.4 0.4)
+				(thickness 0.1)
+			)
+			(justify left bottom mirror)
+		)
+	)
+	(gr_text "OUT"
+		(at 124.9 90.4 0)
+		(layer "B.SilkS")
+		(effects
+			(font
+				(size 1 1)
+				(thickness 0.1)
+			)
+			(justify left bottom mirror)
+		)
+	)
 	(segment
 		(start 122.165 103)
@@
 	)
 	(segment
+		(start 125.22 98.67)
+		(end 122.165 101.725)
+		(width 1)
+		(layer "F.Cu")
+		(net 5)
+	)
+	(segment
 		(start 127.499999 107.132499)
 		(end 127.78 107.4125)
@@
 	)
 	(segment
-		(start 122.165 101.725)
-		(end 124.699804 99.190196)
-		(width 1)
-		(layer "F.Cu")
-		(net 5)
-	)
-	(segment
 		(start 125.5 107.4125)
 		(end 130.32 107.4125)
@@
 	)
 	(segment
-		(start 124.699804 99.190196)
-		(end 125.22 98.67)
-		(width 1)
-		(layer "F.Cu")
-		(net 5)
-	)
-	(segment
 		(start 125.24 106.075)
 		(end 125.24 107.4125)
@@
 	)
 	(segment
+		(start 127.475 101.675276)
+		(end 127.500001 101.700277)
+		(width 1)
+		(layer "F.Cu")
+		(net 6)
+	)
+	(segment
+		(start 127.475 99.225)
+		(end 127.475 101.675276)
+		(width 1)
+		(layer "F.Cu")
+		(net 6)
+	)
+	(segment
 		(start 117.835 107.1975)
 		(end 117.62 107.4125)
@@
 	)
 	(segment
+		(start 127.45 99.2)
+		(end 127.475 99.225)
+		(width 1)
+		(layer "F.Cu")
+		(net 6)
+	)
+	(segment
 		(start 117.835 103)
 		(end 117.835 107.1975)
@@
 		(net 6)
 	)
-	(segment
-		(start 129.78 98.67)
-		(end 128.33 98.67)
-		(width 1)
-		(layer "F.Cu")
-		(net 6)
-	)
-	(segment
-		(start 127.500001 101.700277)
-		(end 127.5 99.5)
-		(width 1)
-		(layer "F.Cu")
-		(net 6)
-	)
-	(segment
-		(start 128.33 98.67)
-		(end 127.5 99.5)
-		(width 1)
-		(layer "F.Cu")
-		(net 6)
-	)
 	(via
-		(at 127.5 99.5)
+		(at 129.775 89.9)
 		(size 1.2)
 		(drill 0.3)
@@
 		(net 6)
 	)
+	(via
+		(at 125.25 94.1)
+		(size 1.2)
+		(drill 0.3)
+		(layers "F.Cu" "B.Cu")
+		(free yes)
+		(net 6)
+	)
+	(via
+		(at 127.5 91.875)
+		(size 1.2)
+		(drill 0.3)
+		(layers "F.Cu" "B.Cu")
+		(free yes)
+		(net 6)
+	)
+	(via
+		(at 127.45 99.2)
+		(size 1.2)
+		(drill 0.3)
+		(layers "F.Cu" "B.Cu")
+		(free yes)
+		(net 6)
+	)
+	(via
+		(at 125.225 89.9)
+		(size 1.2)
+		(drill 0.3)
+		(layers "F.Cu" "B.Cu")
+		(free yes)
+		(net 6)
+	)
+	(via
+		(at 129.775 94.125)
+		(size 1.2)
+		(drill 0.3)
+		(layers "F.Cu" "B.Cu")
+		(free yes)
+		(net 6)
+	)
 	(segment
 		(start 125.24 87.369606)
@@
 	)
 	(segment
+		(start 117.475 96.325)
+		(end 117.475 95.925)
+		(width 1)
+		(layer "F.Cu")
+		(net 7)
+	)
+	(segment
 		(start 121.9 91.5)
 		(end 121.9 90.709606)
@@
 	)
 	(segment
-		(start 117.5 97)
-		(end 117.5 95.9)
-		(width 1)
-		(layer "F.Cu")
-		(net 7)
-	)
-	(segment
 		(start 125.24 86.6625)
 		(end 130.32 86.6625)
@@
 	)
 	(segment
-		(start 117.5 95.9)
-		(end 121.9 91.5)
-		(width 1)
-		(layer "F.Cu")
-		(net 7)
-	)
-	(segment
 		(start 122.2 91.5)
 		(end 122.9425 91.5)
@@
 	)
 	(segment
+		(start 117.475 95.925)
+		(end 121.9 91.5)
+		(width 1)
+		(layer "F.Cu")
+		(net 7)
+	)
+	(segment
 		(start 121.9 90.709606)
 		(end 125.24 87.369606)
@@
 	)
 	(segment
-		(start 122.5 97)
-		(end 127.5 92)
+		(start 129.78 97.63)
+		(end 128.425 96.275)
 		(width 1)
 		(layer "F.Cu")
@@
 	)
 	(segment
-		(start 121.5 97)
-		(end 122.5 97)
-		(width 1)
-		(layer "F.Cu")
+		(start 128.375 96.325)
+		(end 121.475 96.325)
+		(width 1)
+		(layer "F.Cu")
+		(net 8)
+	)
+	(segment
+		(start 129.78 98.67)
+		(end 129.78 97.63)
+		(width 1)
+		(layer "F.Cu")
+		(net 8)
+	)
+	(segment
+		(start 128.425 96.275)
+		(end 128.375 96.325)
+		(width 1)
+		(layer "F.Cu")

Commit message: Added more vias to U1 GND pad for stability
Routing:
- net GNDPWR: vias 6 -> 10
Changed lines of the file:
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@@
+	)
+	(via
+		(at 127.5 94.1)
+		(size 1.2)
+		(drill 0.3)
+		(layers "F.Cu" "B.Cu")
+		(free yes)
+		(net 6)
+	)
+	(via
+		(at 125.25 91.875)
+		(size 1.2)
+		(drill 0.3)
+		(layers "F.Cu" "B.Cu")
+		(free yes)
+		(net 6)
 	)
 	(via
 		(at 129.775 89.9)
+		(size 1.2)
+		(drill 0.3)
+		(layers "F.Cu" "B.Cu")
+		(free yes)
+		(net 6)
+	)
+	(via
+		(at 127.5 89.9)
 		(size 1.2)
 		(drill 0.3)
@@
 		(size 1.2)
 		(drill 0.3)
+		(layers "F.Cu" "B.Cu")
+		(free yes)
+		(net 6)
+	)
+	(via
+		(at 129.775 92)
+		(size 1.2)
+		(drill 0.3)

Commit message: Updated silk screen info
Other:
- board text added: "Nanoka DC-DC Module Input: 6v min, 25v max Output: 5v @ 1A max"
- board text removed: "Nanoka DC-DC Module Input: 6v min, 2Ov max Output: 5v @ 1.5A max"
Changed lines of the file:
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@@
 		(layer "Edge.Cuts")
 	)
-	(gr_text "Nanoka DC-DC Module\nInput: 6v min, 2Ov max\nOutput: 5v @ 1.5A max "
+	(gr_text "Nanoka DC-DC Module\nInput: 6v min, 25v max\nOutput: 5v @ 1A max "
 		(at 127.35 98.225 0)
 		(layer "B.SilkS")

Commit message: Updated schematic to be much clearer
Parts:
- D2: value TVS 29.2V -> SMBJ36A
Connections:
- net Net-(D1-K) renamed OUT+
- net Net-(D2-K) renamed IN+
Changed lines of the file:
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@@
 	(net 3 "unconnected-(J2-Pin_7-Pad7)")
 	(net 4 "unconnected-(J2-Pin_6-Pad6)")
-	(net 5 "Net-(D2-K)")
+	(net 5 "IN+")
 	(net 6 "GNDPWR")
-	(net 7 "Net-(D1-K)")
+	(net 7 "OUT+")
 	(net 8 "Net-(D1-A)")
 	(footprint "Custom:PinHeader_1x12_P1.27mm_Vertical_Modded"
@@
 			(layers "*.Cu" "*.Mask")
 			(remove_unused_layers no)
-			(net 5 "Net-(D2-K)")
+			(net 5 "IN+")
 			(pinfunction "Pin_8")
 			(pintype "passive")
@@
 			(layers "*.Cu" "*.Mask")
 			(remove_unused_layers no)
-			(net 5 "Net-(D2-K)")
+			(net 5 "IN+")
 			(pinfunction "Pin_9")
 			(pintype "passive")
@@
 			(layers "*.Cu" "*.Mask")
 			(remove_unused_layers no)
-			(net 5 "Net-(D2-K)")
+			(net 5 "IN+")
 			(pinfunction "Pin_10")
 			(pintype "passive")
@@
 			(layers "*.Cu" "*.Mask")
 			(remove_unused_layers no)
-			(net 5 "Net-(D2-K)")
+			(net 5 "IN+")
 			(pinfunction "Pin_11")
 			(pintype "passive")
@@
 			(layers "*.Cu" "*.Mask")
 			(remove_unused_layers no)
-			(net 5 "Net-(D2-K)")
+			(net 5 "IN+")
 			(pinfunction "Pin_12")
 			(pintype "passive")
@@
 			)
 		)
-		(property "Value" "TVS 29.2V"
+		(property "Value" "SMBJ36A"
 			(at 2.945 3.0625 0)
 			(layer "F.Fab")
@@
 			(size 2.28 2.12)
 			(layers "F.Cu" "F.Mask" "F.Paste")
-			(net 5 "Net-(D2-K)")
+			(net 5 "IN+")
 			(pinfunction "K")
 			(pintype "passive")
@@
 			(size 0.98 2.4)
 			(layers "F.Cu" "F.Mask" "F.Paste")
-			(net 5 "Net-(D2-K)")
+			(net 5 "IN+")
 			(pinfunction "IN")
 			(pintype "power_in")
@@
 			(size 3 1.6)
 			(layers "F.Cu" "F.Mask" "F.Paste")
-			(net 7 "Net-(D1-K)")
+			(net 7 "OUT+")
 			(pintype "passive")
 			(solder_mask_margin 0.102)
@@
 			(size 2.299995 1.405349)
 			(layers "F.Cu" "F.Mask" "F.Paste")
-			(net 5 "Net-(D2-K)")
+			(net 5 "IN+")
 			(pintype "passive")
 		)
@@
 			(layers "F.Cu" "F.Mask" "F.Paste")
 			(roundrect_rratio 0.1388888889)
-			(net 7 "Net-(D1-K)")
+			(net 7 "OUT+")
 			(pinfunction "K")
 			(pintype "passive")
@@
 			(layers "*.Cu" "*.Mask")
 			(remove_unused_layers no)
-			(net 7 "Net-(D1-K)")
+			(net 7 "OUT+")
 			(pinfunction "Pin_8")
 			(pintype "passive")
@@
 			(layers "*.Cu" "*.Mask")
 			(remove_unused_layers no)
-			(net 7 "Net-(D1-K)")
+			(net 7 "OUT+")
 			(pinfunction "Pin_9")
 			(pintype "passive")
@@
 			(layers "*.Cu" "*.Mask")
 			(remove_unused_layers no)
-			(net 7 "Net-(D1-K)")
+			(net 7 "OUT+")
 			(pinfunction "Pin_10")
 			(pintype "passive")
@@
 			(layers "*.Cu" "*.Mask")
 			(remove_unused_layers no)
-			(net 7 "Net-(D1-K)")
+			(net 7 "OUT+")
 			(pinfunction "Pin_11")
 			(pintype "passive")
@@
 			(layers "*.Cu" "*.Mask")
 			(remove_unused_layers no)
-			(net 7 "Net-(D1-K)")
+			(net 7 "OUT+")
 			(pinfunction "Pin_12")
 			(pintype "passive")

Commit message: Complete re-design
Parts:
- added C4: 33uf, Footprints2:C_1206_3216Metric, F.Cu at (127.5, 90.5)
- added C5: 33uf, Footprints2:C_1206_3216Metric, F.Cu at (130.0, 90.5)
- added C6: 33uf, Footprints2:C_1206_3216Metric, F.Cu at (119.5, 90.5)
- added C7: 33uf, Footprints2:C_1206_3216Metric, F.Cu at (117.0, 90.5)
- added R1: 400, Footprints2:R_1206_3216Metric, F.Cu at (117.5, 101.0)
- C1: footprint Custom:CAPMP3.7X2.8_2.1N_KEM -> Footprints2:C_1206_3216Metric
- C2: value 330mf -> 10uf; footprint Custom:CAP_20SVPK68M -> Footprints2:C_1206_3216Metric
- D1: footprint Diode_SMD:D_SMA -> Footprints2:D_SMA
- D2: value SMBJ36A -> LED; footprint Custom:DIOM4336X265N -> Footprints2:LED_0805_2012Metric
- J1, J2: footprint Custom:PinHeader_1x12_P1.27mm_Vertical_Modded -> Footprints2:PinHeader_1x12_P1.27mm_Vertical_Modded
- U1: value L7805 -> TPS7B8650DQDDARQ1; footprint Custom:VREG_L7805CDT-TR -> Footprints2:DDA0008B-IPC_B
- moved C2 11.5 mm to (128.0, 99.5)
- moved U1 8.77 mm to (123.0, 102.0), turned to -90 degrees
- moved D2 6.18 mm to (118.5, 97.0), turned to 0 degrees
- moved D1 5.91 mm to (123.5, 92.0), turned to -90 degrees
- moved C1 1.58 mm to (128.0, 104.5), turned to 180 degrees
Connections:
- C1 pad 1: IN+ -> GNDPWR
- C1 pad 2: GNDPWR -> IN+
- C2 pad 1: OUT+ -> GNDPWR
- C2 pad 2: GNDPWR -> Net-(D1-A)
- D2 pad 1: IN+ -> Net-(D2-K)
- D2 pad 2: GNDPWR -> Net-(D1-A)
- U1 pad 1: IN+ -> Net-(D1-A)
- U1 pad 2: Net-(D1-A) -> unconnected-(U1-NC-Pad2)
- U1 pad 3: GNDPWR -> unconnected-(U1-NC-Pad3)
Routing:
- net IN+: track 19.8 -> 12.1 mm
- net OUT+: track 18.7 -> 23.9 mm
- net Net-(D1-A): track 9.93 -> 13.1 mm
- net Net-(D2-K): track 0.00 -> 2.56 mm
- net GNDPWR: track 12.4 -> 9.99 mm, vias 10 -> 14
- added copper zone on F.Cu, net GNDPWR
Other:
- board text added: "+5V"
- board text added: "Nanoka DC-DC Module Input: 6v min, 40v max Output: 5v @ 500mah max"
- board text removed: "Nanoka DC-DC Module Input: 6v min, 25v max Output: 5v @ 1A max"

Commit message: Added central IC 3d model
Routing:
- net OUT+: track 23.9 -> 23.3 mm
Other:
- board text added: "Nanoka DC-DC Module Input: 6v min, 40v max Output: 5v @ 500mA max"
- board text removed: "Nanoka DC-DC Module Input: 6v min, 40v max Output: 5v @ 500mah max"
Changed lines of the file:
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@@
 		)
 		(embedded_fonts no)
+		(model "${KIPRJMOD}/assets/3d_models/DDA0008E.stp"
+			(offset
+				(xyz 0 0 0)
+			)
+			(scale
+				(xyz 1 1 1)
+			)
+			(rotate
+				(xyz 0 0 0)
+			)
+		)
 	)
 	(gr_poly
@@
 		)
 	)
-	(gr_text "Nanoka DC-DC Module\nInput: 6v min, 40v max\nOutput: 5v @ 500mah max"
+	(gr_text "Nanoka DC-DC Module\nInput: 6v min, 40v max\nOutput: 5v @ 500mA max"
 		(at 127 92.5 0)
 		(layer "B.SilkS")
@@
 		(layer "F.Cu")
 		(net 7)
-	)
-	(segment
-		(start 129.5 87.1125)
-		(end 129.05 86.6625)
-		(width 0.5)
-		(layer "F.Cu")
-		(net 7)
