File: PowerMod.kicad_pcb (KiCad board)
At the start: 2 copper layers, 16.2 x 23.8 mm, 7 parts, among them J1 Conn_01x12_Pin, J2 Conn_01x12_Pin, U1 L7805

Commit message: Embedded symbols and footprints
Other:
- board text added: "Nanoka DC-DC Module Input: 6v min, 30v max Output: 5v @ 1A max"
- board text removed: "Nanoka DC-DC Module Input: 6v min, 25v max Output: 5v @ 1A max"
Changed lines of the file:
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@@
 		(layer "Edge.Cuts")
 	)
-	(gr_text "Nanoka DC-DC Module\nInput: 6v min, 25v max\nOutput: 5v @ 1A max "
+	(gr_text "Nanoka DC-DC Module\nInput: 6v min, 30v max\nOutput: 5v @ 1A max "
 		(at 127.35 98.225 0)
 		(layer "B.SilkS")
